File: boards/base_v2_lite/base_v2_lite.kicad_sch (KiCad schematic)
At the start: 27 parts, among them J1 Hexpansion-Connector, U2 CH32V006F8Ux

Commit message: Replace base symbol after library renames
Parts:
- J1: footprint tildagon:hexpansion-edge-connector -> matrix-hexpansion:hexpansion-edge-connector; symbol hexpansion-adapter:hexpansion-edge-connector -> matrix-hexpansion:hexpansion-edge-connector
- J3: symbol hexpansion-adapter:hexpansion-adapter-lite -> matrix-hexpansion:matrix-hexpansion-base-v2; now in the parts list
Changed lines of the file:
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@@
 	)
 	(symbol
-		(lib_id "hexpansion-adapter:hexpansion-adapter-lite")
+		(lib_id "matrix-hexpansion:matrix-hexpansion-base-v2")
 		(at 176.53 120.65 0)
 		(unit 1)
 		(body_style 1)
 		(exclude_from_sim no)
-		(in_bom no)
+		(in_bom yes)
 		(on_board yes)
 		(in_pos_files yes)
@@
 	)
 	(symbol
-		(lib_id "hexpansion-adapter:hexpansion-edge-connector")
+		(lib_id "matrix-hexpansion:hexpansion-edge-connector")
 		(at 36.83 46.99 0)
 		(unit 1)
@@
 			)
 		)
-		(property "Footprint" "tildagon:hexpansion-edge-connector"
+		(property "Footprint" "matrix-hexpansion:hexpansion-edge-connector"
 			(at 36.83 49.53 0)
 			(hide yes)
@@
 			)
 		)
-		(property "Datasheet" ""
+		(property "Datasheet" "https://www.wch-ic.com/products/CH32V003.html"
 			(at 147.32 46.99 0)
 			(hide yes)
