File: boards/base_v2_lite/base_v2_lite.kicad_pcb (KiCad board)
At the start: 2 copper layers, 40 x 34 mm, 31 parts, among them J1 Hexpansion-Connector, U2 CH32V006F8Ux

Commit message: Replace base symbol after library renames
Parts:
- J1: footprint tildagon:hexpansion-edge-connector -> matrix-hexpansion:hexpansion-edge-connector
Changed lines of the file:
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@@
 		(embedded_fonts no)
 	)
-	(footprint "tildagon:hexpansion-edge-connector"
+	(footprint "matrix-hexpansion:hexpansion-edge-connector"
 		(layer "F.Cu")
 		(at 120 62 -90)
@@
 				(font
 					(size 1.27 1.27)
+					(thickness 0.15)
 				)
 			)
@@
 				(font
 					(size 1.27 1.27)
+					(thickness 0.15)
 				)
 			)
@@
 			)
 		)
-		(property "Datasheet" ""
+		(property "Datasheet" "https://www.wch-ic.com/products/CH32V003.html"
 			(at 0 0 0)
 			(layer "F.Fab")
@@
 			)
 		)
-		(attr exclude_from_bom)
 		(duplicate_pad_numbers_are_jumpers no)
 		(fp_line

Commit message: Remove KiKit markers, add license to base silkscreen
Parts:
- removed REF** (x4): Tab, PCM_kikit:Tab
Other:
- board text added: "License: CERN-OHL-W"
- board text added: "base v2.2 2026-08-30 5yk.de"
- board text removed: "base v2.1 lite 2026-08-27"
