File: boards/lite_loop/lite_loop.kicad_pcb (KiCad board)
At the start: 2 copper layers, 71.4 x 31 mm, 173 parts

Commit message: Remove KiKit markers, add license to base silkscreen
Parts:
- removed REF** (x3): Tab, PCM_kikit:Tab
Other:
- board text added: "5yk.de/matrix-hexpansion/lite-loop 2026-08-30"
- board text removed: "5yk.de/matrix-hexpansion/lite-loop 2026-07-25"
